File: .history/Project Architecture.kicad_sch (KiCad schematic)
At the start: 0 parts

Commit message: Schematic changes done
Other:
- sheet Section A - Title A renamed Section A - MCU
- removed sheet Section B - Title B
- added sheet Power Section (Power Section.kicad_sch)
- sheet Section A - MCU: file Section A - Title A.kicad_sch -> Section A - MCU.kicad_sch
- note removed: "Page 5"
Changed lines of the file:
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@@
-	)
-	(arc
-		(start 234.97 124.44)
-		(mid 234.0749 124.0651)
-		(end 233.7 123.17)
-		(stroke
-			(width 0)
-			(type default)
-		)
-		(fill
-			(type none)
-		)
-	)
-	(arc
-		(start 233.7 125.71)
-		(mid 234.0749 124.8149)
-		(end 234.97 124.44)
-		(stroke
-			(width 0)
-			(type default)
-		)
-		(fill
-			(type none)
-		)
-	)
-	(arc
-		(start 233.7 134.6)
-		(mid 232.9561 136.3961)
-		(end 231.16 137.14)
-		(stroke
-			(width 0)
-			(type default)
-		)
-		(fill
-			(type none)
-		)
 	)
 	(arc
@@
 	)
 	(arc
-		(start 231.16 111.74)
-		(mid 232.9502 112.4898)
-		(end 233.7 114.28)
-		(stroke
-			(width 0)
-			(type default)
-		)
-		(fill
-			(type none)
-		)
-	)
-	(arc
 		(start 185.42 73.66)
 		(mid 186.1639 71.8639)
@@
 		(fill
 			(type none)
-		)
-	)
-	(text "Page 5"
-		(exclude_from_sim no)
-		(at 226.06 133.35 0)
-		(effects
-			(font
-				(size 2.54 2.54)
-				(bold yes)
-				(color 100 70 50 1)
-			)
-			(justify right bottom)
-			(href "#5")
 		)
 	)
@@
 		)
 	)
-	(text_box "Description"
-		(exclude_from_sim no)
-		(at 234.95 121.92 0)
-		(size 26.015 5.1)
-		(margins 1.4287 1.4287 1.4287 1.4287)
-		(stroke
-			(width -0.0001)
-			(type default)
-		)
-		(fill
-			(type none)
-		)
-		(effects
-			(font
-				(size 1.905 1.905)
-				(thickness 0.381)
-				(bold yes)
-				(color 0 0 0 1)
-			)
-			(justify left top)
-		)
-	)
 	(text_box "[${#}] ${TITLE}"
 		(exclude_from_sim no)
@@
 	(polyline
 		(pts
-			(xy 233.68 125.73) (xy 233.68 134.62)
-		)
-		(stroke
-			(width 0)
-			(type default)
-		)
-	)
-	(polyline
-		(pts
 			(xy 185.42 85.09) (xy 185.42 73.66)
 		)
@@
 		)
 	)
-	(polyline
-		(pts
-			(xy 233.68 114.3) (xy 233.68 123.19)
-		)
-		(stroke
-			(width 0)
-			(type default)
-		)
-	)
 	(sheet
-		(at 190.5 114.3)
-		(size 36.83 20.32)
+		(at 116.84 74.93)
+		(size 36.83 22.86)
 		(exclude_from_sim no)
 		(in_bom yes)
@@
 		)
 		(fill
-			(color 255 200 0 0.502)
+			(color 0 0 0 0)
 		)
-		(property "Sheetname" "Section B - Title B"
-			(at 190.5 113.2709 0)
+		(property "Sheetname" "Power Section"
+			(at 116.84 74.2184 0)
 			(show_name no)
 			(do_not_autoplace no)
 			(effects
 				(font
-					(size 1.905 1.905)
-					(bold yes)
+					(size 1.27 1.27)
 				)
 				(justify left bottom)
 			)
 		)
-		(property "Sheetfile" "Section B - TItle B.kicad_sch"
-			(at 190.5 135.2046 0)
+		(property "Sheetfile" "Power Section.kicad_sch"
+			(at 116.84 98.3746 0)
 			(show_name no)
 			(do_not_autoplace no)
 			(effects
 				(font
-					(face "Arial")
 					(size 1.27 1.27)
 				)
@@
 			(project "KiBot_Project_Test"
 				(path "/f9e05184-c88b-4a88-ae9c-ab2bdb32be7c/c5103ceb-5325-4a84-a025-9638a412984e"
-					(page "5")
+					(page "8")
 				)
 			)
@@
 			(color 128 255 128 0.5)
 		)
-		(property "Sheetname" "Section A - Title A"
+		(property "Sheetname" "Section A - MCU"
 			(at 190.5 75.1709 0)
 			(show_name no)
@@
 			)
 		)
-		(property "Sheetfile" "Section A - Title A.kicad_sch"
+		(property "Sheetfile" "Section A - MCU.kicad_sch"
 			(at 190.5 97.1046 0)
 			(show_name no)
